Commit message: 从官方示例项目中拆解基础框架，调整参数适应我们的gazebo中ur5机械臂的视觉抓取。已经成功运行显示，下一步为添加摄像头组件。

File: urdf/ur5_with_camera.urdf.xacro (robot description, xacro)
@@ -1,98 +1,86 @@
 <?xml version="1.0"?>
-<robot xmlns:xacro="http://www.ros.org/wiki/xacro" name="ur5_with_camera">
-  <!-- 直接包含底层宏文件 -->
-  <xacro:include filename="$(find ur_description)/urdf/ur_macro.xacro" />
-  <!-- 定义摄像头参数 -->
-  <xacro:arg name="camera_width" default="640"/>
-  <xacro:arg name="camera_height" default="480"/>
-  <xacro:arg name="camera_fps" default="30"/>
-  <xacro:arg name="camera_name" default="camera"/>
-  <!-- 定义world链接 -->
-  <link name="world" />
-  <!-- 实例化UR5机械臂 -->
-  <xacro:ur_robot
-    name="ur5"
-    tf_prefix=""
-    parent="world"
-    joint_limits_parameters_file="$(find ur_description)/config/ur5/joint_limits.yaml"
-    kinematics_parameters_file="$(find ur_description)/config/ur5/default_kinematics.yaml"
-    physical_parameters_file="$(find ur_description)/config/ur5/physical_parameters.yaml"
-    visual_parameters_file="$(find ur_description)/config/ur5/visual_parameters.yaml"
-    safety_limits="true"
-    safety_pos_margin="0.15"
-    safety_k_position="20"
-  >
-    <origin xyz="0 0 0" rpy="0 0 0" />
-  </xacro:ur_robot>
-  <!-- 在末端添加摄像头 -->
-  <!-- ✅ 修正：使用 $(arg camera_name) 而不是 ${camera_name} -->
-  <link name="$(arg camera_name)_link">
-    <visual>
-      <geometry>
-        <box size="0.03 0.03 0.01"/>
-      </geometry>
-      <material name="black">
-        <color rgba="0.1 0.1 0.1 1.0"/>
-      </material>
-    </visual>
-    <collision>
-      <geometry>
-        <box size="0.03 0.03 0.01"/>
-      </geometry>
-    </collision>
-    <inertial>
-      <mass value="0.01"/>
-      <inertia ixx="1e-6" ixy="0" ixz="0" iyy="1e-6" iyz="0" izz="1e-6"/>
-    </inertial>
-  </link>
-  <!-- ✅ 修正：使用 $(arg camera_name) -->
-  <joint name="$(arg camera_name)_joint" type="fixed">
-    <parent link="tool0"/>
-    <child link="$(arg camera_name)_link"/>
-    <origin xyz="0.0 0.0 0.02" rpy="0 ${pi/2} 0"/>
-  </joint>
-  <!-- ✅ 修正：使用 $(arg camera_name) -->
-  <gazebo reference="$(arg camera_name)_link">
-    <material>Gazebo/Black</material>
-  </gazebo>
-  <!-- ✅ 修正：使用 $(arg camera_name) -->
-  <gazebo reference="$(arg camera_name)_link">
-    <sensor type="camera" name="$(arg camera_name)">
-      <update_rate>$(arg camera_fps)</update_rate>
-      <camera name="head">
-        <horizontal_fov>1.0471975512</horizontal_fov>
-        <image>
-          <width>$(arg camera_width)</width>
-          <height>$(arg camera_height)</height>
-          <format>R8G8B8</format>
-        </image>
-        <clip>
-          <near>0.02</near>
-          <far>300</far>
-        </clip>
-        <noise>
-          <type>gaussian</type>
-          <mean>0.0</mean>
-          <stddev>0.007</stddev>
-        </noise>
-      </camera>
-      <plugin filename="libgazebo_ros_camera.so" name="$(arg camera_name)_controller">
-        <ros>
-          <namespace>$(arg camera_name)</namespace>
-          <remapping>~/image_raw:=image_raw</remapping>
-          <remapping>~/camera_info:=camera_info</remapping>
-        </ros>
-        <camera_name>$(arg camera_name)</camera_name>
-        <frame_name>$(arg camera_name)_link</frame_name>
-        <hack_baseline>0.07</hack_baseline>
+<robot xmlns:xacro="http://wiki.ros.org/xacro" name="$(arg name)">
+   <!-- robot name parameter -->
+   <xacro:arg name="name" default="ur"/>
+   <!-- import main macro -->
+   <xacro:include filename="$(find ur_description)/urdf/ur_macro.xacro"/>
+   <!-- possible 'ur_type' values: ur3, ur5, ur10, ur3e, ur5e, ur7e, ur10e, ur12e, ur16e, ur8long, ur15, ur18, ur20, ur30 -->
+   <!-- the default value should raise an error in case this was called without defining the type -->
+   <xacro:arg name="ur_type" default="ur5"/>
+   <!-- parameters that need to be configurable -->
+   <xacro:arg name="tf_prefix" default="" />
+   <xacro:arg name="safety_limits" default="true"/>
+   <!-- Simulation parameters -->
+   <xacro:arg name="sim_gazebo" default="true" />
+   <xacro:arg name="sim_ignition" default="false" />
+   <xacro:arg name="simulation_controllers" default="$(find ur_simulation_gazebo)/config/ur_controllers.yaml" />
+   <!-- initial position for simulations (Fake Hardware, Gazebo, Ignition) -->
+   <xacro:arg name="initial_positions_file" default="$(find ur_description)/config/initial_positions.yaml"/>
+   <!-- convert to property to use substitution in function -->
+   <xacro:property name="initial_positions_file" default="$(arg initial_positions_file)"/>
+   <xacro:property name="is_sim_gazebo" value="$(arg sim_gazebo)"/>
+   <xacro:property name="is_sim_ignition" value="$(arg sim_ignition)"/>
+   <!-- create link fixed to the "world" -->
+   <link name="world" />
+   <xacro:if value="${is_sim_gazebo or is_sim_ignition}">
+     <link name="ground_plane">
+       <visual>
+         <origin rpy="0 0 0" xyz="0 0 0"/>
+         <geometry>
+           <box size="5 5 0"/>
+         </geometry>
+         <material name="ground_white">
+           <color rgba="1 1 1 0.5"/>
+         </material>
+       </visual>
+       <collision>
+         <origin rpy="0 0 0" xyz="0 0 0"/>
+         <geometry>
+           <box size="5 5 0"/>
+         </geometry>
+       </collision>
+     </link>
+     <joint name="ground_plane_joint" type="fixed">
+       <origin xyz="0 0 -0.01" rpy="0 0 0"/>
+       <parent link="world"/>
+       <child link="ground_plane"/>
+     </joint>
+   </xacro:if>
+   <!-- arm -->
+   <xacro:ur_robot
+     name="$(arg name)"
+     tf_prefix="$(arg tf_prefix)"
+     parent="world"
+     joint_limits_parameters_file="$(find ur_description)/config/$(arg ur_type)/joint_limits.yaml"
+     kinematics_parameters_file="$(find ur_description)/config/$(arg ur_type)/default_kinematics.yaml"
+     physical_parameters_file="$(find ur_description)/config/$(arg ur_type)/physical_parameters.yaml"
+     visual_parameters_file="$(find ur_description)/config/$(arg ur_type)/visual_parameters.yaml"
+     safety_limits="$(arg safety_limits)"
+     sim_gazebo="$(arg sim_gazebo)"
+     sim_ignition="$(arg sim_ignition)"
+     initial_positions="${xacro.load_yaml(initial_positions_file)}"
+     >
+     <origin xyz="0 0 0" rpy="0 0 0" />          <!-- position robot in the world -->
+   </xacro:ur_robot>
+   <xacro:if value="$(arg sim_gazebo)">
+    <!-- Gazebo plugins -->
+    <gazebo reference="world">
+    </gazebo>
+    <gazebo>
+      <plugin filename="libgazebo_ros2_control.so" name="gazebo_ros2_control">
+        <parameters>$(arg simulation_controllers)</parameters>
       </plugin>
-    </sensor>
-  </gazebo>
-  <gazebo>
-    <light type="point" name="point_light">
-      <pose>0 0 3 0 0 0</pose>
-      <diffuse>0.8 0.8 0.8 1</diffuse>
-      <specular>0.2 0.2 0.2 1</specular>
-    </light>
-  </gazebo>
+    </gazebo>
+  </xacro:if>
+  <xacro:if value="$(arg sim_ignition)">
+    <!-- Gazebo plugins -->
+    <gazebo reference="world">
+    </gazebo>
+    <gazebo>
+      <plugin filename="libign_ros2_control-system.so" name="ign_ros2_control::IgnitionROS2ControlPlugin">
+        <parameters>$(arg simulation_controllers)</parameters>
+        <controller_manager_node_name>$(arg tf_prefix)controller_manager</controller_manager_node_name>
+      </plugin>
+    </gazebo>
+  </xacro:if>
 </robot>

Commit message: 添加摄像头：分清摄像头坐标系和光学坐标系对图像和算法的影响。添加rviz配置文件，集中显示。

File: urdf/ur5_with_camera.urdf.xacro (robot description, xacro)
@@ -63,4 +63,77 @@
      <origin xyz="0 0 0" rpy="0 0 0" />          <!-- position robot in the world -->
    </xacro:ur_robot>
+   <!-- Camera joint - connected to tool0 -->
+   <joint name="camera_joint" type="fixed">
+     <origin xyz="0.0 0.0 0.015" rpy="0 -1.570796 1.570796"/>
+     <parent link="tool0"/>
+     <child link="camera_link"/>
+   </joint>
+   <!-- Camera link -->
+   <link name="camera_link">
+     <visual>
+       <origin xyz="0 0 0" rpy="0 0 0"/>
+       <geometry>
+         <box size="0.02 0.02 0.02"/>
+       </geometry>
+       <material name="red">
+         <color rgba="1 0 0 1"/>
+       </material>
+     </visual>
+     <collision>
+       <origin xyz="0 0 0" rpy="0 0 0"/>
+       <geometry>
+         <box size="0.02 0.02 0.02"/>
+       </geometry>
+     </collision>
+     <inertial>
+       <mass value="0.1"/>
+       <origin xyz="0 0 0" rpy="0 0 0"/>
+       <inertia ixx="0.0001" ixy="0" ixz="0" iyy="0.0001" iyz="0" izz="0.0001"/>
+     </inertial>
+   </link>
+   <!-- Gazebo material for camera link -->
+   <gazebo reference="camera_link">
+     <material>Gazebo/Red</material>
+   </gazebo>
+   <!-- Camera optical joint -->
+   <joint name="camera_optical_joint" type="fixed">
+     <origin xyz="0 0 0" rpy="-1.570796 0 -1.570796"/>
+     <parent link="camera_link"/>
+     <child link="camera_link_optical"/>
+   </joint>
+   <!-- Camera optical link -->
+   <link name="camera_link_optical"></link>
+   <!-- Gazebo camera plugin -->
+   <gazebo reference="camera_link">
+     <sensor type="camera" name="camera">
+       <update_rate>30.0</update_rate>
+       <camera name="head">
+         <horizontal_fov>1.3962634</horizontal_fov>
+         <image>
+           <width>800</width>
+           <height>600</height>
+           <format>R8G8B8</format>
+         </image>
+         <clip>
+           <near>0.02</near>
+           <far>300</far>
+         </clip>
+         <noise>
+           <type>gaussian</type>
+           <mean>0.0</mean>
+           <stddev>0.007</stddev>
+         </noise>
+       </camera>
+       <plugin name="camera_controller" filename="libgazebo_ros_camera.so">
+         <alwaysOn>true</alwaysOn>
+         <updateRate>0.0</updateRate>
+         <cameraName>camera</cameraName>
+         <imageTopicName>image_raw</imageTopicName>
+         <cameraInfoTopicName>camera_info</cameraInfoTopicName>
+         <frameName>camera_link_optical</frameName>
+         <hackBaseline>0.07</hackBaseline>
+       </plugin>
+     </sensor>
+   </gazebo>
    <xacro:if value="$(arg sim_gazebo)">
     <!-- Gazebo plugins -->

Commit message: opence物体识别：红色正方体。光照阴影所需的hsv调整。

File: urdf/ur5_with_camera.urdf.xacro (robot description, xacro)
@@ -16,5 +16,5 @@
    <xacro:arg name="simulation_controllers" default="$(find ur_simulation_gazebo)/config/ur_controllers.yaml" />
    <!-- initial position for simulations (Fake Hardware, Gazebo, Ignition) -->
-   <xacro:arg name="initial_positions_file" default="$(find ur_description)/config/initial_positions.yaml"/>
+   <xacro:arg name="initial_positions_file" default="$(find vision_grasp_demo)/config/initial_positions.yaml"/>
    <!-- convert to property to use substitution in function -->
    <xacro:property name="initial_positions_file" default="$(arg initial_positions_file)"/>
@@ -65,5 +65,5 @@
    <!-- Camera joint - connected to tool0 -->
    <joint name="camera_joint" type="fixed">
-     <origin xyz="0.0 0.0 0.015" rpy="0 -1.570796 1.570796"/>
+     <origin xyz="0.0 0.0 0.03" rpy="1.570796 0 0"/>
      <parent link="tool0"/>
      <child link="camera_link"/>
